File: Dynakku.kicad_sch (KiCad schematic)
At the start: 12 parts, among them J1 Conn_01x02, Q1 CSD17577Q3A

Commit message: dev
Parts:
- renumbered D3 to D2, D2 to D3, D6 to D5, D5 to D6, R2 to R1, R1 to R2
Changed lines of the file:
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@@
 		(in_pos_files yes)
 		(dnp no)
-		(property "Reference" "#PWR06"
+		(property "Reference" "#PWR03"
 			(at 92.71 57.15 0)
 			(hide yes)
@@
 			(project "Dynakku"
 				(path "/a6a976ba-6389-49ad-86f2-b30a2d1aab45"
-					(reference "#PWR06")
+					(reference "#PWR03")
 					(unit 1)
 				)
@@
 		(in_pos_files yes)
 		(dnp no)
-		(property "Reference" "R1"
+		(property "Reference" "R2"
 			(at 97.028 75.946 0)
 			(show_name no)
@@
 			(project "Dynakku"
 				(path "/a6a976ba-6389-49ad-86f2-b30a2d1aab45"
-					(reference "R1")
+					(reference "R2")
 					(unit 1)
 				)
@@
 		(in_pos_files yes)
 		(dnp no)
-		(property "Reference" "D2"
+		(property "Reference" "D3"
 			(at 71.12 29.21 0)
 			(show_name no)
@@
 			(project "Dynakku"
 				(path "/a6a976ba-6389-49ad-86f2-b30a2d1aab45"
-					(reference "D2")
+					(reference "D3")
 					(unit 1)
 				)
@@
 		(in_pos_files yes)
 		(dnp no)
-		(property "Reference" "#PWR05"
+		(property "Reference" "#PWR06"
 			(at 113.03 66.04 0)
 			(hide yes)
@@
 			(project "Dynakku"
 				(path "/a6a976ba-6389-49ad-86f2-b30a2d1aab45"
-					(reference "#PWR05")
+					(reference "#PWR06")
 					(unit 1)
 				)
@@
 		(in_pos_files yes)
 		(dnp no)
-		(property "Reference" "D6"
+		(property "Reference" "D5"
 			(at 95.25 59.436 90)
 			(show_name no)
@@
 			(project "Dynakku"
 				(path "/a6a976ba-6389-49ad-86f2-b30a2d1aab45"
-					(reference "D6")
+					(reference "D5")
 					(unit 1)
 				)
@@
 		(in_pos_files yes)
 		(dnp no)
-		(property "Reference" "#PWR03"
+		(property "Reference" "#PWR04"
 			(at 92.71 88.9 0)
 			(hide yes)
@@
 			(project "Dynakku"
 				(path "/a6a976ba-6389-49ad-86f2-b30a2d1aab45"
-					(reference "#PWR03")
+					(reference "#PWR04")
 					(unit 1)
 				)
@@
 		(dnp no)
 		(fields_autoplaced yes)
-		(property "Reference" "D5"
+		(property "Reference" "D6"
 			(at 96.8375 38.1 0)
 			(show_name no)
@@
 			(project "Dynakku"
 				(path "/a6a976ba-6389-49ad-86f2-b30a2d1aab45"
-					(reference "D5")
+					(reference "D6")
 					(unit 1)
 				)
@@
 		(in_pos_files yes)
 		(dnp no)
-		(property "Reference" "R2"
-			(at 94.488 68.58 0)
+		(property "Reference" "R1"
+			(at 94.488 66.548 0)
 			(show_name no)
 			(do_not_autoplace no)
@@
 		)
 		(property "Value" "1k"
-			(at 94.488 66.04 0)
+			(at 94.742 68.58 0)
 			(show_name no)
 			(do_not_autoplace no)
@@
 			(project "Dynakku"
 				(path "/a6a976ba-6389-49ad-86f2-b30a2d1aab45"
-					(reference "R2")
+					(reference "R1")
 					(unit 1)
 				)
@@
 		(in_pos_files yes)
 		(dnp no)
-		(property "Reference" "D3"
+		(property "Reference" "D2"
 			(at 53.34 39.116 0)
 			(show_name no)
@@
 			(project "Dynakku"
 				(path "/a6a976ba-6389-49ad-86f2-b30a2d1aab45"
-					(reference "D3")
+					(reference "D2")
 					(unit 1)
 				)
@@
 		(dnp no)
 		(fields_autoplaced yes)
-		(property "Reference" "#PWR04"
+		(property "Reference" "#PWR05"
 			(at 113.03 43.18 0)
 			(hide yes)
@@
 			(project "Dynakku"
 				(path "/a6a976ba-6389-49ad-86f2-b30a2d1aab45"
-					(reference "#PWR04")
-					(unit 1)
-				)
+					(reference "#PWR05")
+					(unit 1)
+				)

Commit message: dev
Parts:
- D1, D2, D3, D4, D6: value 1N5819HW -> SS34
- R1: value 1k -> 2.2k
Changed lines of the file:
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@@
 			)
 		)
-		(property "Value" "1N5819HW"
+		(property "Value" "SS34"
 			(at 71.12 31.75 0)
 			(show_name no)
@@
 			)
 		)
-		(property "Value" "1N5819HW"
+		(property "Value" "SS34"
 			(at 53.34 31.75 0)
 			(show_name no)
@@
 			)
 		)
-		(property "Value" "1N5819HW"
+		(property "Value" "SS34"
 			(at 96.8375 40.64 0)
 			(show_name no)
@@
 			)
 		)
-		(property "Value" "1k"
+		(property "Value" "2.2k"
 			(at 94.742 68.58 0)
 			(show_name no)
@@
 			)
 		)
-		(property "Value" "1N5819HW"
+		(property "Value" "SS34"
 			(at 53.34 41.656 0)
 			(show_name no)
@@
 			)
 		)
-		(property "Value" "1N5819HW"
+		(property "Value" "SS34"
 			(at 71.12 41.656 0)
 			(show_name no)

Commit message: assigned most footprints, changed Input Cap. for charge controller.
Parts:
- removed J1: Conn_01x02, symbol Connector_Generic:Conn_01x02
- added J1, J2: Conn_01x01_Pin, TestPoint:TestPoint_Pad_D3.0mm, symbol Connector:Conn_01x01_Pin
- D1, D2, D3, D4, D6: footprint (none) -> Diode_SMD:D_SMC_Handsoldering
- D5: footprint Package_TO_SOT_SMD:SOT-23 -> Package_TO_SOT_SMD:SOT-23_Handsoldering
- Q1: footprint (none) -> Package_SON:VSONP-8-1EP_5x6_P1.27mm
- R1, R2: footprint (none) -> Resistor_SMD:R_0603_1608Metric_Pad0.98x0.95mm_HandSolder
Connections:
- net AC+: now reaches C1.1
- net AC+: now also J1.1 (Pin_1)
- net AC-: now reaches D2.1 (K), D4.2 (A)
- net AC-: now also J2.1 (Pin_1)
Other:
- moved on the sheet: C1, C2, D1, D2, D3, D4, D5, D6, Q1, R1, R2
