File: battery_protection.kicad_sch (KiCad schematic)
At the start: 6 parts, among them Q4 CSD17577Q3A, Q5 CSD17577Q3A, U2 BQ29700

Commit message: yes
Changed lines of the file:
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@@
 		(in_pos_files yes)
 		(dnp no)
-		(fields_autoplaced yes)
 		(property "Reference" "U2"
-			(at 45.72 20.32 0)
+			(at 45.72 21.336 0)
 			(show_name no)
 			(do_not_autoplace no)
@@
 		)
 		(property "Value" "BQ29700"
-			(at 45.72 22.86 0)
+			(at 45.72 23.876 0)
 			(show_name no)
 			(do_not_autoplace no)
