File: interfaces.kicad_sch (KiCad schematic)
At the start: 7 parts, among them J2 USB_C_Receptacle_PowerOnly_24P, J3 Conn_01x01_Pin, J4 Conn_01x01_Pin

Commit message: dev
Connections:
- net USB_SHIELD is gone; now on net GND: J2.SH (SHIELD)
Changed lines of the file:
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@@
+	(wire
+		(pts
+			(xy 125.73 91.44) (xy 125.73 97.79)
+		)
+		(stroke
+			(width 0)
+			(type default)
+		)
+	)
 	(wire
 		(pts
@@
 		(pts
 			(xy 50.8 95.25) (xy 50.8 99.06)
+		)
+		(stroke
+			(width 0)
+			(type default)
+		)
+	)
+	(wire
+		(pts
+			(xy 114.3 91.44) (xy 125.73 91.44)
 		)
 		(stroke
@@
 	(label "USB_CC2"
 		(at 58.42 110.49 0)
+		(effects
+			(font
+				(size 1.27 1.27)
+			)
+			(justify left bottom)
+		)
+	)
+	(label "USB_SHIELD"
+		(at 114.3 91.44 0)
 		(effects
 			(font
@@
 		(dnp no)
 		(fields_autoplaced yes)
-		(property "Reference" "#PWR042"
+		(property "Reference" "#PWR039"
 			(at 25.4 114.3 0)
 			(hide yes)
@@
 			(project "Dynakku"
 				(path "/c789b728-e330-430f-b4c1-34535a34c880"
-					(reference "#PWR042")
+					(reference "#PWR039")
+					(unit 1)
+				)
+			)
+		)
+	)
+	(symbol
+		(lib_id "power:GND")
+		(at 125.73 97.79 0)
+		(unit 1)
+		(body_style 1)
+		(exclude_from_sim no)
+		(in_bom yes)
+		(on_board yes)
+		(in_pos_files yes)
+		(dnp no)
+		(fields_autoplaced yes)
+		(property "Reference" "#PWR046"
+			(at 125.73 104.14 0)
+			(hide yes)
+			(show_name no)
+			(do_not_autoplace no)
+			(effects
+				(font
+					(size 1.27 1.27)
+				)
+			)
+		)
+		(property "Value" "GND"
+			(at 125.73 102.87 0)
+			(show_name no)
+			(do_not_autoplace no)
+			(effects
+				(font
+					(size 1.27 1.27)
+				)
+			)
+		)
+		(property "Footprint" ""
+			(at 125.73 97.79 0)
+			(hide yes)
+			(show_name no)
+			(do_not_autoplace no)
+			(effects
+				(font
+					(size 1.27 1.27)
+				)
+			)
+		)
+		(property "Datasheet" ""
+			(at 125.73 97.79 0)
+			(hide yes)
+			(show_name no)
+			(do_not_autoplace no)
+			(effects
+				(font
+					(size 1.27 1.27)
+				)
+			)
+		)
+		(property "Description" "Power symbol creates a global label with name \"GND\" , ground"
+			(at 125.73 97.79 0)
+			(hide yes)
+			(show_name no)
+			(do_not_autoplace no)
+			(effects
+				(font
+					(size 1.27 1.27)
+				)
+			)
+		)
+		(pin "1"
+		)
+		(instances
+			(project "Dynakku"
+				(path "/c789b728-e330-430f-b4c1-34535a34c880"
+					(reference "#PWR046")
 					(unit 1)
 				)
@@
 		(dnp no)
 		(fields_autoplaced yes)
-		(property "Reference" "#PWR038"
+		(property "Reference" "#PWR042"
 			(at 90.17 99.06 0)
 			(hide yes)
@@
 			(project "Dynakku"
 				(path "/c789b728-e330-430f-b4c1-34535a34c880"
-					(reference "#PWR038")
+					(reference "#PWR042")
 					(unit 1)
 				)
@@
 		(dnp no)
 		(fields_autoplaced yes)
-		(property "Reference" "#PWR039"
+		(property "Reference" "#PWR043"
 			(at 106.68 104.14 0)
 			(hide yes)
@@
 			(project "Dynakku"
 				(path "/c789b728-e330-430f-b4c1-34535a34c880"
-					(reference "#PWR039")
+					(reference "#PWR043")
 					(unit 1)
 				)
@@
 		(dnp no)
 		(fields_autoplaced yes)
-		(property "Reference" "#PWR043"
+		(property "Reference" "#PWR038"
 			(at 25.4 99.06 0)
 			(hide yes)
@@
 			(project "Dynakku"
 				(path "/c789b728-e330-430f-b4c1-34535a34c880"
-					(reference "#PWR043")
+					(reference "#PWR038")
 					(unit 1)
 				)

Commit message: assigned most footprints, changed Input Cap. for charge controller.
Parts:
- F1: footprint (none) -> Fuse:Fuse_1206_3216Metric_Pad1.42x1.75mm_HandSolder
- J4: renamed from J3; footprint (none) -> TestPoint:TestPoint_Pad_D3.0mm
- J5: renamed from J4; footprint (none) -> TestPoint:TestPoint_Pad_D3.0mm
- R16, R17: footprint (none) -> Resistor_SMD:R_0603_1608Metric_Pad0.98x0.95mm_HandSolder
- renumbered J2 to J3
Changed lines of the file:
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@@
 		(dnp no)
 		(fields_autoplaced yes)
-		(property "Reference" "J4"
+		(property "Reference" "J5"
 			(at 86.995 41.91 0)
 			(show_name no)
@@
 			)
 		)
-		(property "Footprint" ""
+		(property "Footprint" "TestPoint:TestPoint_Pad_D3.0mm"
 			(at 86.36 46.99 0)
 			(hide yes)
@@
 			(project "Dynakku"
 				(path "/c789b728-e330-430f-b4c1-34535a34c880"
-					(reference "J4")
+					(reference "J5")
 					(unit 1)
 				)
@@
 		(dnp no)
 		(fields_autoplaced yes)
-		(property "Reference" "J2"
+		(property "Reference" "J3"
 			(at 36.83 25.4 0)
 			(show_name no)
@@
 			(project "Dynakku"
 				(path "/c789b728-e330-430f-b4c1-34535a34c880"
-					(reference "J2")
+					(reference "J3")
 					(unit 1)
 				)
@@
 			)
 		)
-		(property "Footprint" ""
+		(property "Footprint" "Resistor_SMD:R_0603_1608Metric_Pad0.98x0.95mm_HandSolder"
 			(at 49.022 102.87 90)
 			(hide yes)
@@
 		(dnp no)
 		(fields_autoplaced yes)
-		(property "Reference" "J3"
+		(property "Reference" "J4"
 			(at 86.995 33.02 0)
 			(show_name no)
@@
 			)
 		)
-		(property "Footprint" ""
+		(property "Footprint" "TestPoint:TestPoint_Pad_D3.0mm"
 			(at 86.36 38.1 0)
 			(hide yes)
@@
 			(project "Dynakku"
 				(path "/c789b728-e330-430f-b4c1-34535a34c880"
-					(reference "J3")
+					(reference "J4")
 					(unit 1)
 				)
@@
 			)
 		)
-		(property "Footprint" ""
+		(property "Footprint" "Resistor_SMD:R_0603_1608Metric_Pad0.98x0.95mm_HandSolder"
 			(at 65.532 102.87 90)
 			(hide yes)
@@
 			)
 		)
-		(property "Footprint" ""
+		(property "Footprint" "Fuse:Fuse_1206_3216Metric_Pad1.42x1.75mm_HandSolder"
 			(at 100.33 39.878 90)
 			(hide yes)
