File: mppt_charger.kicad_sch (KiCad schematic)
At the start: 23 parts, among them Q2 CSD17577Q3A, Q3 CSD17577Q3A, U1 BQ24650

Commit message: dev
Parts:
- renumbered C9 to C10, C10 to C11, C5 to C3, C3 to C4, C4 to C5, C7 to C6, C6 to C7, C11 to C8, C8 to C9, R12 to R10, R13 to R11, R5 to R3, R6 to R4, R7 to R5, R8 to R6, R9 to R7, R10 to R8, R11 to R9

Commit message: dev
Parts:
- D7: value 1N5819HW -> SS34
Changed lines of the file:
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@@
 			)
 		)
-		(property "Value" "1N5819HW"
+		(property "Value" "SS34"
 			(at 125.73 120.3324 90)
 			(show_name no)

Commit message: assigned most footprints, changed Input Cap. for charge controller.
Parts:
- added C10, C9: 1µ 50V, Capacitor_SMD:C_0805_2012Metric_Pad1.18x1.45mm_HandSolder, symbol Device:C
- C11: renamed from C9; footprint (none) -> Capacitor_SMD:C_0603_1608Metric_Pad1.08x0.95mm_HandSolder
- C12: renamed from C10; value 10µ 35V -> 10µ 16V; footprint (none) -> Capacitor_SMD:C_0805_2012Metric_Pad1.18x1.45mm_HandSolder
- C13: renamed from C11; value 10µ 35V -> 10µ 16V; footprint (none) -> Capacitor_SMD:C_0805_2012Metric_Pad1.18x1.45mm_HandSolder
- C3, C5, C7: footprint (none) -> Capacitor_SMD:C_0805_2012Metric_Pad1.18x1.45mm_HandSolder
- C4, C6: footprint (none) -> Capacitor_SMD:C_0603_1608Metric_Pad1.08x0.95mm_HandSolder
- C8: value 10µ 35V -> 1µ 50V; footprint (none) -> Capacitor_SMD:C_0805_2012Metric_Pad1.18x1.45mm_HandSolder
- D7: footprint (none) -> Diode_SMD:D_SMC_Handsoldering
- Q2, Q3: footprint (none) -> Package_SON:VSONP-8-1EP_5x6_P1.27mm
- R10, R11, R3, R4, R5, R6, R7, R8, R9: footprint (none) -> Resistor_SMD:R_0603_1608Metric_Pad0.98x0.95mm_HandSolder
Connections:
- net GND: now also C10.2, C9.2
- net VDC: now also C10.1, C9.1
