File: usb_boost.kicad_sch (KiCad schematic)
At the start: 8 parts, among them U3 TPS61022

Commit message: assigned most footprints, changed Input Cap. for charge controller.
Parts:
- C15: renamed from C13; value 10µ 35V -> 10µ 16V; footprint (none) -> Capacitor_SMD:C_0805_2012Metric_Pad1.18x1.45mm_HandSolder
- C16: renamed from C14; value 10µ 35V -> 10µ 16V; footprint (none) -> Capacitor_SMD:C_0805_2012Metric_Pad1.18x1.45mm_HandSolder
- C17: renamed from C15; value 10µ 35V -> 10µ 16V; footprint (none) -> Capacitor_SMD:C_0805_2012Metric_Pad1.18x1.45mm_HandSolder
- C18: renamed from C16; value 10µ 35V -> 10µ 16V; footprint (none) -> Capacitor_SMD:C_0805_2012Metric_Pad1.18x1.45mm_HandSolder
- R14, R15: footprint (none) -> Resistor_SMD:R_0603_1608Metric_Pad0.98x0.95mm_HandSolder
Changed lines of the file:
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@@
 			)
 		)
-		(property "Footprint" ""
+		(property "Footprint" "Resistor_SMD:R_0603_1608Metric_Pad0.98x0.95mm_HandSolder"
 			(at 150.622 82.55 90)
 			(hide yes)
@@
 		(in_pos_files yes)
 		(dnp no)
-		(property "Reference" "C13"
+		(property "Reference" "C15"
 			(at 40.64 88.8999 0)
 			(show_name no)
@@
 			)
 		)
-		(property "Value" "10µ 35V"
+		(property "Value" "10µ 16V"
 			(at 40.64 91.4399 0)
 			(show_name no)
@@
 			)
 		)
-		(property "Footprint" ""
+		(property "Footprint" "Capacitor_SMD:C_0805_2012Metric_Pad1.18x1.45mm_HandSolder"
 			(at 39.0652 93.98 0)
 			(hide yes)
@@
 			(project "Dynakku"
 				(path "/ae2c3cd8-d75c-4533-b378-e05723f24e06"
-					(reference "C13")
+					(reference "C15")
 					(unit 1)
 				)
@@
 		(in_pos_files yes)
 		(dnp no)
-		(property "Reference" "C15"
+		(property "Reference" "C17"
 			(at 80.264 82.55 0)
 			(show_name no)
@@
 			)
 		)
-		(property "Value" "10µ 35V"
+		(property "Value" "10µ 16V"
 			(at 80.264 85.09 0)
 			(show_name no)
@@
 			)
 		)
-		(property "Footprint" ""
+		(property "Footprint" "Capacitor_SMD:C_0805_2012Metric_Pad1.18x1.45mm_HandSolder"
 			(at 78.4352 87.63 0)
 			(hide yes)
@@
 			(project "Dynakku"
 				(path "/ae2c3cd8-d75c-4533-b378-e05723f24e06"
-					(reference "C15")
+					(reference "C17")
 					(unit 1)
 				)
@@
 			)
 		)
-		(property "Footprint" ""
+		(property "Footprint" "Resistor_SMD:R_0603_1608Metric_Pad0.98x0.95mm_HandSolder"
 			(at 150.622 95.25 90)
 			(hide yes)
@@
 		(in_pos_files yes)
 		(dnp no)
-		(property "Reference" "C16"
+		(property "Reference" "C18"
 			(at 95.504 82.55 0)
 			(show_name no)
@@
 			)
 		)
-		(property "Value" "10µ 35V"
+		(property "Value" "10µ 16V"
 			(at 95.504 85.09 0)
 			(show_name no)
@@
 			)
 		)
-		(property "Footprint" ""
+		(property "Footprint" "Capacitor_SMD:C_0805_2012Metric_Pad1.18x1.45mm_HandSolder"
 			(at 93.6752 87.63 0)
 			(hide yes)
@@
 			(project "Dynakku"
 				(path "/ae2c3cd8-d75c-4533-b378-e05723f24e06"
-					(reference "C16")
+					(reference "C18")
 					(unit 1)
 				)
@@
 		(in_pos_files yes)
 		(dnp no)
-		(property "Reference" "C14"
+		(property "Reference" "C16"
 			(at 65.024 82.55 0)
 			(show_name no)
@@
 			)
 		)
-		(property "Value" "10µ 35V"
+		(property "Value" "10µ 16V"
 			(at 65.024 85.09 0)
 			(show_name no)
@@
 			)
 		)
-		(property "Footprint" ""
+		(property "Footprint" "Capacitor_SMD:C_0805_2012Metric_Pad1.18x1.45mm_HandSolder"
 			(at 63.1952 87.63 0)
 			(hide yes)
@@
 			(project "Dynakku"
 				(path "/ae2c3cd8-d75c-4533-b378-e05723f24e06"
-					(reference "C14")
-					(unit 1)
-				)
+					(reference "C16")
+					(unit 1)
+				)
