File: Dynakku.kicad_pcb (KiCad board)
At the start: 4 copper layers, 40 x 60 mm, 60 parts, among them J1 Conn_01x01_Pin, J2 Conn_01x01_Pin, J4 Conn_01x01_Pin, J5 Conn_01x01_Pin, J6 UJC-V-G-SMT-P6-TR, Q1 CSD17577Q3A, Q2 CSD17577Q3A, Q3 CSD17577Q3A, Q4 CSD17577Q3A, Q5 CSD17577Q3A, U1 BQ24650, U2 BQ29700, U3 TPS61022

Commit message: yes
Parts:
- moved C5 0.17 mm to (113.1, 74.8)
- moved C7 0.17 mm to (111.0, 74.8)
- moved C9 0.17 mm to (106.8, 74.8)
- moved C8 0.17 mm to (108.9, 74.8)
Routing:
- net /MPPT Charger/BQ24650_REGN: track 0.00 -> 7.84 mm, vias 0 -> 2
- net VDC: track 15.9 -> 23.4 mm
- net /MPPT Charger/BQ24650_HIDRV: track 1.66 -> 6.79 mm, vias 1 -> 0
- net /MPPT Charger/BQ24650_VREF: track 3.95 -> 7.93 mm
- net /MPPT Charger/BQ24650_VFB: track 8.51 -> 9.30 mm
Changed lines of the file:
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@@
 	(footprint "Capacitor_SMD:C_0805_2012Metric_Pad1.18x1.45mm_HandSolder"
 		(layer "B.Cu")
-		(at 111.175 74.8375 90)
+		(at 111.004803 74.839803 90)
 		(descr "Capacitor SMD 0805 (2012 Metric), square (rectangular) end terminal, IPC-7351 nominal with elongated pad for handsoldering. (Body size source: IPC-SM-782 page 76, https://www.pcb-3d.com/wordpress/wp-content/uploads/ipc-sm-782a_amendment_1_and_2.pdf, https://docs.google.com/spreadsheets/d/1BsfQQcO9C6DZCsRaXUlFlo91Tg2WpOkGARC1WS5S8t0/edit?usp=sharing)")
 		(tags "capacitor handsolder")
@@
 	(footprint "Capacitor_SMD:C_0805_2012Metric_Pad1.18x1.45mm_HandSolder"
 		(layer "B.Cu")
-		(at 113.275 74.8375 90)
+		(at 113.104803 74.839803 90)
 		(descr "Capacitor SMD 0805 (2012 Metric), square (rectangular) end terminal, IPC-7351 nominal with elongated pad for handsoldering. (Body size source: IPC-SM-782 page 76, https://www.pcb-3d.com/wordpress/wp-content/uploads/ipc-sm-782a_amendment_1_and_2.pdf, https://docs.google.com/spreadsheets/d/1BsfQQcO9C6DZCsRaXUlFlo91Tg2WpOkGARC1WS5S8t0/edit?usp=sharing)")
 		(tags "capacitor handsolder")
@@
 	(footprint "Capacitor_SMD:C_0805_2012Metric_Pad1.18x1.45mm_HandSolder"
 		(layer "B.Cu")
-		(at 109.1 74.8375 90)
+		(at 108.929803 74.839803 90)
 		(descr "Capacitor SMD 0805 (2012 Metric), square (rectangular) end terminal, IPC-7351 nominal with elongated pad for handsoldering. (Body size source: IPC-SM-782 page 76, https://www.pcb-3d.com/wordpress/wp-content/uploads/ipc-sm-782a_amendment_1_and_2.pdf, https://docs.google.com/spreadsheets/d/1BsfQQcO9C6DZCsRaXUlFlo91Tg2WpOkGARC1WS5S8t0/edit?usp=sharing)")
 		(tags "capacitor handsolder")
@@
 	(footprint "Capacitor_SMD:C_0805_2012Metric_Pad1.18x1.45mm_HandSolder"
 		(layer "B.Cu")
-		(at 107.01 74.8375 90)
+		(at 106.839803 74.839803 90)
 		(descr "Capacitor SMD 0805 (2012 Metric), square (rectangular) end terminal, IPC-7351 nominal with elongated pad for handsoldering. (Body size source: IPC-SM-782 page 76, https://www.pcb-3d.com/wordpress/wp-content/uploads/ipc-sm-782a_amendment_1_and_2.pdf, https://docs.google.com/spreadsheets/d/1BsfQQcO9C6DZCsRaXUlFlo91Tg2WpOkGARC1WS5S8t0/edit?usp=sharing)")
 		(tags "capacitor handsolder")
@@
 	)
 	(via
-		(at 107.35 72.55)
+		(at 107.225 72.55)
 		(size 0.6)
 		(drill 0.3)
@@
 	)
 	(via
-		(at 106.625 72.55)
+		(at 106.5 72.55)
 		(size 0.6)
 		(drill 0.3)
@@
 	)
 	(via
-		(at 111.575 72.575)
+		(at 111.45 72.575)
 		(size 0.6)
 		(drill 0.3)
@@
 	)
 	(via
-		(at 108.725 72.575)
+		(at 108.6 72.575)
 		(size 0.6)
 		(drill 0.3)
@@
 	)
 	(via
-		(at 113.75 72.575)
+		(at 113.625 72.575)
 		(size 0.6)
 		(drill 0.3)
@@
 	)
 	(via
-		(at 109.45 72.575)
+		(at 109.325 72.575)
 		(size 0.6)
 		(drill 0.3)
@@
 	)
 	(via
-		(at 113.025 72.575)
+		(at 112.9 72.575)
 		(size 0.6)
 		(drill 0.3)
@@
 	)
 	(via
-		(at 110.85 72.575)
+		(at 110.725 72.575)
 		(size 0.6)
 		(drill 0.3)
@@
 	)
 	(segment
-		(start 114.375 76.9125)
-		(end 114.375 76.7)
+		(start 114.104606 74.864803)
+		(end 109.942303 74.864803)
 		(width 0.25)
 		(layer "B.Cu")
@@
 	)
 	(segment
-		(start 90.5 77.5)
-		(end 90.5 76.75)
+		(start 109.942303 74.864803)
+		(end 108.929803 75.877303)
 		(width 0.25)
 		(layer "B.Cu")
@@
 	)
 	(segment
+		(start 90.5 77.5)
+		(end 90.5 76.75)
+		(width 0.25)
+		(layer "B.Cu")
+		(net "VDC")
+	)
+	(segment
+		(start 114.375 75.135197)
+		(end 114.104606 74.864803)
+		(width 0.25)
+		(layer "B.Cu")
+		(net "VDC")
+	)
+	(segment
+		(start 114.375 76.9125)
+		(end 114.375 75.135197)
+		(width 0.25)
+		(layer "B.Cu")
+		(net "VDC")
+	)
+	(segment
 		(start 100.75 59)
 		(end 103.5 61.75)
@@
 	)
 	(segment
-		(start 101.911602 79.275)
-		(end 100.2645 80.922102)
+		(start 100.2645 80.922102)
+		(end 100.2645 83.550666)
 		(width 0.2)
 		(layer "B.Cu")
@@
 	)
 	(segment
-		(start 107.75 77.855)
-		(end 107.5225 78.0825)
+		(start 97.0545 83.9245)
+		(end 96.25 83.12)
 		(width 0.2)
 		(layer "B.Cu")
@@
 	)
 	(segment
-		(start 100.2645 80.922102)
-		(end 100.2645 83.550666)
+		(start 107.605 78)
+		(end 104.5 78)
 		(width 0.2)
 		(layer "B.Cu")
@@
 	)
 	(segment
-		(start 106.580614 78.0825)
-		(end 105.388114 79.275)
+		(start 99.890666 83.9245)
+		(end 97.0545 83.9245)
 		(width 0.2)
 		(layer "B.Cu")
@@
 	)
 	(segment
-		(start 105.388114 79.275)
+		(start 103.225 79.275)
 		(end 101.911602 79.275)
 		(width 0.2)
@@
 	)
 	(segment
-		(start 100.2645 83.550666)
-		(end 99.890666 83.9245)
+		(start 104.5 78)
+		(end 103.225 79.275)
 		(width 0.2)
 		(layer "B.Cu")
@@
 	)
 	(segment
-		(start 99.890666 83.9245)
-		(end 97.0545 83.9245)
+		(start 107.75 77.855)
+		(end 107.605 78)
 		(width 0.2)
 		(layer "B.Cu")
@@
 	)
 	(segment
-		(start 107.5225 78.0825)
-		(end 106.580614 78.0825)
+		(start 100.2645 83.550666)
+		(end 99.890666 83.9245)
 		(width 0.2)
 		(layer "B.Cu")
@@
 	)
 	(segment
-		(start 97.0545 83.9245)
-		(end 96.25 83.12)
+		(start 101.911602 79.275)
+		(end 100.2645 80.922102)
 		(width 0.2)
 		(layer "B.Cu")
@@
 	)
 	(segment
-		(start 108.75 81.691886)
-		(end 109.035614 81.9775)
+		(start 109.625 86.2875)
+		(end 109.625 82.566886)
 		(width 0.2)
 		(layer "B.Cu")
@@
 	)
 	(segment
-		(start 109.5525 81.9775)
-		(end 109.7975 82.2225)
+		(start 109.425 86.4875)
+		(end 109.625 86.2875)
 		(width 0.2)
 		(layer "B.Cu")
@@
 	)
 	(segment
-		(start 108.75 81.25)
-		(end 108.75 81.691886)
+		(start 110.4125 86.4875)
+		(end 110.525 86.6)
 		(width 0.2)
 		(layer "B.Cu")
@@
 	)
 	(segment
-		(start 110.4125 86.4875)
-		(end 110.525 86.6)
+		(start 109.625 82.566886)
+		(end 108.75 81.691886)
 		(width 0.2)
 		(layer "B.Cu")
@@
 	)
 	(segment
-		(start 109.035614 81.9775)
-		(end 109.5525 81.9775)
+		(start 108.75 81.691886)
+		(end 108.75 81.25)
 		(width 0.2)
 		(layer "B.Cu")
@@
 	)
 	(segment
-		(start 111.275 81.375)
-		(end 111.275 83.370642)
+		(start 110.1975 80.303826)
+		(end 111.250774 81.3571)
 		(width 0.2)
 		(layer "B.Cu")
@@
 	)
 	(segment
-		(start 111.3 83.395642)
+		(start 111.250774 85.500774)
 		(end 111.3 85.55)
 		(width 0.2)
@@
 	)
 	(segment
-		(start 111.275 83.370642)
-		(end 111.3 83.395642)
+		(start 111.250774 81.3571)
+		(end 111.250774 85.500774)
 		(width 0.2)
 		(layer "B.Cu")
@@
 	)
 	(segment
-		(start 110.2025 80.3025)
-		(end 111.275 81.375)
+		(start 111.5875 85.55)
+		(end 112.9 86.8625)
 		(width 0.2)
 		(layer "B.Cu")
@@
 	)
 	(segment
-		(start 111.5875 85.55)
-		(end 112.9 86.8625)
+		(start 110.1975 80.3025)
+		(end 110.1975 80.303826)
 		(width 0.2)
 		(layer "B.Cu")
@@
 	)
 	(segment
-		(start 110.1975 80.3025)
-		(end 110.2025 80.3025)
+		(start 110 77)
+		(end 107 77)
+		(width 0.2)
+		(layer "F.Cu")
+		(net "/MPPT Charger/BQ24650_REGN")
+	)
+	(segment
+		(start 105.8025 78.1975)
+		(end 105.8025 78.8025)
+		(width 0.2)
+		(layer "F.Cu")
+		(net "/MPPT Charger/BQ24650_REGN")
+	)
+	(segment
+		(start 107 77)
+		(end 105.8025 78.1975)
+		(width 0.2)
+		(layer "F.Cu")
+		(net "/MPPT Charger/BQ24650_REGN")
+	)
+	(via
+		(at 110 77)
+		(size 0.6)
+		(drill 0.3)
+		(layers "F.Cu" "B.Cu")
+		(net "/MPPT Charger/BQ24650_REGN")
+	)
+	(via
+		(at 105.8025 78.8025)
+		(size 0.6)
+		(drill 0.3)
+		(layers "F.Cu" "B.Cu")
+		(net "/MPPT Charger/BQ24650_REGN")
+	)
+	(segment
+		(start 105.8025 78.8025)
+		(end 106.8025 78.8025)
 		(width 0.2)
 		(layer "B.Cu")
-		(net "/MPPT Charger/BQ24650_TS")
+		(net "/MPPT Charger/BQ24650_REGN")
+	)
+	(segment
+		(start 111.004803 75.995197)
+		(end 110 77)
+		(width 0.2)
+		(layer "B.Cu")
+		(net "/MPPT Charger/BQ24650_REGN")
+	)
+	(segment
+		(start 111.004803 75.877303)
+		(end 111.004803 75.995197)
+		(width 0.2)
+		(layer "B.Cu")
+		(net "/MPPT Charger/BQ24650_REGN")
 	)
 	(segment
@@
 	)
 	(segment
-		(start 107.375 83.080033)
-		(end 107.375 87.075)
-		(width 0.2)
-		(layer "F.Cu")
-		(net "/MPPT Charger/BQ24650_VFB")
-	)
-	(segment
-		(start 108.186305 82.227261)
-		(end 108.184681 82.228885)
+		(start 107.619766 82.273373)
+		(end 107.619766 86.847198)
 		(width 0.2)
 		(layer "F.Cu")
@@
 	)
 	(segment
-		(start 107.375 87.075)
+		(start 107.619766 86.847198)
 		(end 107.383482 87.083482)
 		(width 0.2)
@@
 		(net "/MPPT Charger/BQ24650_VFB")
 	)
-	(segment
-		(start 108.184681 82.228885)
-		(end 108.184681 82.270352)
-		(width 0.2)
-		(layer "F.Cu")
-		(net "/MPPT Charger/BQ24650_VFB")
-	)
-	(segment
-		(start 108.184681 82.270352)
-		(end 107.375 83.080033)
-		(width 0.2)
-		(layer "F.Cu")
-		(net "/MPPT Charger/BQ24650_VFB")
-	)
 	(via
-		(at 108.186305 82.227261)
+		(at 107.619766 82.273373)
 		(size 0.6)
 		(drill 0.3)
@@
 	)
 	(segment
+		(start 107.619766 82.273373)
+		(end 107.75 82.143139)
+		(width 0.2)
+		(layer "B.Cu")
+		(net "/MPPT Charger/BQ24650_VFB")
+	)
+	(segment
 		(start 105.5125 88.4875)
 		(end 105.375 88.35)
@@
 	)
 	(segment
+		(start 107.75 82.143139)
+		(end 107.75 81.25)
+		(width 0.2)
+		(layer "B.Cu")
+		(net "/MPPT Charger/BQ24650_VFB")
+	)
+	(segment
 		(start 107.125 88.4875)
 		(end 107.125 87.341964)
@@
 		(net "/MPPT Charger/BQ24650_VCC")
 	)
-	(via
-		(at 109.8 77.1)
-		(size 0.6)
-		(drill 0.3)
-		(layers "F.Cu" "B.Cu")
+	(segment
+		(start 108.201689 76.864803)
+		(end 103.295197 76.864803)
+		(width 0.2)
+		(layer "B.Cu")
 		(net "/MPPT Charger/BQ24650_HIDRV")
 	)
 	(segment
-		(start 109.8 77.1)
-		(end 109 77.1)
+		(start 108.75 77.855)
+		(end 108.75 77.413114)
 		(width 0.2)
 		(layer "B.Cu")
@@
 	)
 	(segment
-		(start 109 77.1)
-		(end 108.75 77.35)
+		(start 108.75 77.413114)
+		(end 108.201689 76.864803)
 		(width 0.2)
 		(layer "B.Cu")
@@
 	)
 	(segment
-		(start 108.75 77.35)
-		(end 108.75 77.855)
+		(start 103.295197 76.864803)
+		(end 102.825 77.335)
 		(width 0.2)
 		(layer "B.Cu")
