File: .history/Dynakku.kicad_sch (KiCad schematic)
At the start: 12 parts, among them J1 Conn_01x02, Q1 CSD17577Q3A

Commit message: assigned most footprints, changed Input Cap. for charge controller.
Parts:
- removed J1: Conn_01x02, symbol Connector_Generic:Conn_01x02
- added J1, J2: Conn_01x01_Pin, TestPoint:TestPoint_Pad_D3.0mm, symbol Connector:Conn_01x01_Pin
- D1, D4: value 1N5819HW -> SS34; footprint (none) -> Diode_SMD:D_SMC_Handsoldering
- D2: renamed from D3; value 1N5819HW -> SS34; footprint (none) -> Diode_SMD:D_SMC_Handsoldering
- D3: renamed from D2; value 1N5819HW -> SS34; footprint (none) -> Diode_SMD:D_SMC_Handsoldering
- D5: renamed from D6; footprint Package_TO_SOT_SMD:SOT-23 -> Package_TO_SOT_SMD:SOT-23_Handsoldering
- D6: renamed from D5; value 1N5819HW -> SS34; footprint (none) -> Diode_SMD:D_SMC_Handsoldering
- Q1: footprint (none) -> Package_SON:VSONP-8-1EP_5x6_P1.27mm
- R1: renamed from R2; value 1k -> 2.2k; footprint (none) -> Resistor_SMD:R_0603_1608Metric_Pad0.98x0.95mm_HandSolder
- R2: renamed from R1; footprint (none) -> Resistor_SMD:R_0603_1608Metric_Pad0.98x0.95mm_HandSolder
Connections:
- net AC+: now reaches C1.1
- net AC+: now also J1.1 (Pin_1)
- net AC-: now reaches D2.1 (K), D4.2 (A)
- net AC-: now also J2.1 (Pin_1)
Other:
- moved on the sheet: C1, C2, D1, D2, D3, D4, D5, D6, Q1, R1, R2

Commit message: Update mcp_config.json, Dynakku.kicad_pcb, Dynakku.kicad_sch, and 20 more files
Parts:
- C1: value 330µ 35V -> ECE-A1HN331U, 330µ 35V; footprint (none) -> Capacitor_THT:C_Radial_D16.0mm_H25.0mm_P7.50mm
- C2: value 1000µ 35V -> UUE1V102MNS6MS, 1000µ 35V; footprint (none) -> Capacitor_SMD:CP_Elec_18x22
- D1, D2, D3, D4, D6: footprint Diode_SMD:D_SMC_Handsoldering -> Diode_SMD:D_SMC
Changed lines of the file:
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@@
 			)
 		)
-		(property "Value" "330µ 35V"
+		(property "Value" "ECE-A1HN331U, 330µ 35V"
 			(at 46.99 22.606 90)
 			(show_name no)
@@
 			)
 		)
-		(property "Footprint" ""
+		(property "Footprint" "Capacitor_THT:C_Radial_D16.0mm_H25.0mm_P7.50mm"
 			(at 50.8 25.7048 0)
 			(hide yes)
@@
 			)
 		)
-		(property "Value" "1000µ 35V"
+		(property "Value" "UUE1V102MNS6MS, 1000µ 35V"
 			(at 119.38 52.4509 0)
 			(show_name no)
@@
 			)
 		)
-		(property "Footprint" ""
+		(property "Footprint" "Capacitor_SMD:CP_Elec_18x22"
 			(at 116.5352 55.88 0)
 			(hide yes)
@@
 			)
 		)
-		(property "Footprint" "Diode_SMD:D_SMC_Handsoldering"
+		(property "Footprint" "Diode_SMD:D_SMC"
 			(at 73.66 34.29 0)
 			(hide yes)
@@
 			)
 		)
-		(property "Footprint" "Diode_SMD:D_SMC_Handsoldering"
+		(property "Footprint" "Diode_SMD:D_SMC"
 			(at 55.88 34.29 0)
 			(hide yes)
@@
 			)
 		)
-		(property "Footprint" "Diode_SMD:D_SMC_Handsoldering"
+		(property "Footprint" "Diode_SMD:D_SMC"
 			(at 99.06 44.45 0)
 			(hide yes)
@@
 			)
 		)
-		(property "Footprint" "Diode_SMD:D_SMC_Handsoldering"
+		(property "Footprint" "Diode_SMD:D_SMC"
 			(at 55.88 44.45 0)
 			(hide yes)
@@
 			)
 		)
-		(property "Footprint" "Diode_SMD:D_SMC_Handsoldering"
+		(property "Footprint" "Diode_SMD:D_SMC"
 			(at 73.66 44.45 0)
 			(hide yes)
