File: .history/battery_protection.kicad_sch (KiCad schematic)
At the start: 6 parts, among them Q4 CSD17577Q3A, Q5 CSD17577Q3A, U2 BQ29700

Commit message: Update mcp_config.json, Dynakku.kicad_pcb, Dynakku.kicad_sch, and 20 more files
Parts:
- C14: value 100n -> 100n 50V
Changed lines of the file:
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@@
 			)
 		)
-		(property "Value" "100n"
+		(property "Value" "100n 50V"
 			(at 29.21 86.3599 0)
 			(show_name no)
