File: .history/interfaces.kicad_sch (KiCad schematic)
At the start: 7 parts, among them J3 USB_C_Receptacle_PowerOnly_24P, J4 Conn_01x01_Pin, J5 Conn_01x01_Pin

Commit message: Update mcp_config.json, Dynakku.kicad_pcb, Dynakku.kicad_sch, and 20 more files
Parts:
- removed J3: USB_C_Receptacle_PowerOnly_24P, symbol Connector:USB_C_Receptacle_PowerOnly_24P
- added J6: UJC-V-G-SMT-P6-TR, UJC-H-G-SMT-2-P6-TR:SAMESKY_UJC-H-G-SMT-2-P6-TR, symbol 2026-07-19_11-56-26:UJC-V-G-SMT-P6-TR
Connections:
- net GND: now also J6.A12 (GND), J6.B12 (GND)
- net USB_CC1: now also J6.A5 (CC1)
- net USB_CC2: now also J6.B5 (CC2)
- net VBUS: now also J6.A9 (VBUS), J6.B9 (VBUS)
