File: .history/mppt_charger.kicad_sch (KiCad schematic)
At the start: 23 parts, among them Q2 CSD17577Q3A, Q3 CSD17577Q3A, U1 BQ24650

Commit message: assigned most footprints, changed Input Cap. for charge controller.
Parts:
- removed C11: 10µ 35V, symbol Device:C
- added C10, C8, C9: 1µ 50V, Capacitor_SMD:C_0805_2012Metric_Pad1.18x1.45mm_HandSolder, symbol Device:C
- C11: renamed from C8; footprint (none) -> Capacitor_SMD:C_0603_1608Metric_Pad1.08x0.95mm_HandSolder
- C12: renamed from C9; value 10µ 35V -> 10µ 16V; footprint (none) -> Capacitor_SMD:C_0805_2012Metric_Pad1.18x1.45mm_HandSolder
- C13: renamed from C10; value 10µ 35V -> 10µ 16V; footprint (none) -> Capacitor_SMD:C_0805_2012Metric_Pad1.18x1.45mm_HandSolder
- C3: renamed from C5; footprint (none) -> Capacitor_SMD:C_0805_2012Metric_Pad1.18x1.45mm_HandSolder
- C4: renamed from C3; footprint (none) -> Capacitor_SMD:C_0603_1608Metric_Pad1.08x0.95mm_HandSolder
- C5: renamed from C4; footprint (none) -> Capacitor_SMD:C_0805_2012Metric_Pad1.18x1.45mm_HandSolder
- C6: renamed from C7; footprint (none) -> Capacitor_SMD:C_0603_1608Metric_Pad1.08x0.95mm_HandSolder
- C7: renamed from C6; footprint (none) -> Capacitor_SMD:C_0805_2012Metric_Pad1.18x1.45mm_HandSolder
- D7: value 1N5819HW -> SS34; footprint (none) -> Diode_SMD:D_SMC_Handsoldering
- Q2, Q3: footprint (none) -> Package_SON:VSONP-8-1EP_5x6_P1.27mm
- R10: renamed from R12; footprint (none) -> Resistor_SMD:R_0603_1608Metric_Pad0.98x0.95mm_HandSolder
- R11: renamed from R13; footprint (none) -> Resistor_SMD:R_0603_1608Metric_Pad0.98x0.95mm_HandSolder
- R3: renamed from R5; footprint (none) -> Resistor_SMD:R_0603_1608Metric_Pad0.98x0.95mm_HandSolder
- R4: renamed from R6; footprint (none) -> Resistor_SMD:R_0603_1608Metric_Pad0.98x0.95mm_HandSolder
- R5: renamed from R7; footprint (none) -> Resistor_SMD:R_0603_1608Metric_Pad0.98x0.95mm_HandSolder
- R6: renamed from R8; footprint (none) -> Resistor_SMD:R_0603_1608Metric_Pad0.98x0.95mm_HandSolder
- R7: renamed from R9; footprint (none) -> Resistor_SMD:R_0603_1608Metric_Pad0.98x0.95mm_HandSolder
- R8: renamed from R10; footprint (none) -> Resistor_SMD:R_0603_1608Metric_Pad0.98x0.95mm_HandSolder
- R9: renamed from R11; footprint (none) -> Resistor_SMD:R_0603_1608Metric_Pad0.98x0.95mm_HandSolder
Connections:
- net GND: now also C10.2, C8.2, C9.2
- net VDC: now also C10.1, C8.1, C9.1

Commit message: Update mcp_config.json, Dynakku.kicad_pcb, Dynakku.kicad_sch, and 20 more files
Parts:
- C11, C4: value 100n -> 100n 50V
- D7: footprint Diode_SMD:D_SMC_Handsoldering -> Diode_SMD:D_SMC
- L1: footprint (none) -> Inductor_SMD:L_Vishay_IHLP-2525
Other:
- moved on the sheet: C4
Changed lines of the file:
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@@
 	(wire
 		(pts
-			(xy 45.72 118.11) (xy 57.15 118.11)
+			(xy 43.18 118.11) (xy 57.15 118.11)
 		)
 		(stroke
@@
 	(wire
 		(pts
-			(xy 45.72 128.27) (xy 45.72 134.62)
+			(xy 43.18 128.27) (xy 43.18 134.62)
 		)
 		(stroke
@@
 	(wire
 		(pts
-			(xy 45.72 118.11) (xy 45.72 120.65)
+			(xy 43.18 118.11) (xy 43.18 120.65)
 		)
 		(stroke
@@
 	(symbol
 		(lib_id "Device:C")
-		(at 45.72 124.46 0)
+		(at 43.18 124.46 0)
 		(unit 1)
 		(body_style 1)
@@
 		(in_pos_files yes)
 		(dnp no)
-		(fields_autoplaced yes)
 		(property "Reference" "C4"
-			(at 49.53 123.1899 0)
+			(at 46.228 123.19 0)
 			(show_name no)
 			(do_not_autoplace no)
@@
 			)
 		)
-		(property "Value" "100n"
-			(at 49.53 125.7299 0)
+		(property "Value" "100n 50V"
+			(at 46.228 125.73 0)
 			(show_name no)
 			(do_not_autoplace no)
@@
 		)
 		(property "Footprint" "Capacitor_SMD:C_0603_1608Metric_Pad1.08x0.95mm_HandSolder"
-			(at 46.6852 128.27 0)
+			(at 44.1452 128.27 0)
 			(hide yes)
 			(show_name no)
@@
 		)
 		(property "Datasheet" ""
-			(at 45.72 124.46 0)
+			(at 43.18 124.46 0)
 			(hide yes)
 			(show_name no)
@@
 		)
 		(property "Description" "Unpolarized capacitor"
-			(at 45.72 124.46 0)
+			(at 43.18 124.46 0)
 			(hide yes)
 			(show_name no)
@@
 		(dnp no)
 		(property "Reference" "C12"
-			(at 216.662 118.11 0)
+			(at 215.392 118.11 0)
 			(show_name no)
 			(do_not_autoplace no)
@@
 	(symbol
 		(lib_id "power:GND")
-		(at 45.72 134.62 0)
+		(at 43.18 134.62 0)
 		(unit 1)
 		(body_style 1)
@@
 		(fields_autoplaced yes)
 		(property "Reference" "#PWR09"
-			(at 45.72 140.97 0)
+			(at 43.18 140.97 0)
 			(hide yes)
 			(show_name no)
@@
 		)
 		(property "Value" "GND"
-			(at 45.72 139.7 0)
+			(at 43.18 139.7 0)
 			(show_name no)
 			(do_not_autoplace no)
@@
 		)
 		(property "Footprint" ""
-			(at 45.72 134.62 0)
+			(at 43.18 134.62 0)
 			(hide yes)
 			(show_name no)
@@
 		)
 		(property "Datasheet" ""
-			(at 45.72 134.62 0)
+			(at 43.18 134.62 0)
 			(hide yes)
 			(show_name no)
@@
 		)
 		(property "Description" "Power symbol creates a global label with name \"GND\" , ground"
-			(at 45.72 134.62 0)
+			(at 43.18 134.62 0)
 			(hide yes)
 			(show_name no)
@@
 			)
 		)
-		(property "Footprint" ""
+		(property "Footprint" "Inductor_SMD:L_Vishay_IHLP-2525"
 			(at 193.04 130.81 0)
 			(hide yes)
@@
 			)
 		)
-		(property "Footprint" "Diode_SMD:D_SMC_Handsoldering"
+		(property "Footprint" "Diode_SMD:D_SMC"
 			(at 123.19 119.38 0)
 			(hide yes)
@@
 		(dnp no)
 		(property "Reference" "C11"
-			(at 196.088 144.78 0)
+			(at 186.436 145.288 0)
 			(show_name no)
 			(do_not_autoplace no)
@@
 			)
 		)
-		(property "Value" "100n"
-			(at 196.088 147.32 0)
+		(property "Value" "100n 50V"
+			(at 180.848 147.32 0)
 			(show_name no)
 			(do_not_autoplace no)
