File: .history/Dynakku.kicad_pcb (KiCad board)
At the start: 4 copper layers, 40 x 60 mm, 59 parts, among them J1 Conn_01x01_Pin, J2 Conn_01x01_Pin, J4 Conn_01x01_Pin, J5 Conn_01x01_Pin, J6 UJC-V-G-SMT-P6-TR, Q1 CSD17577Q3A, Q2 CSD17577Q3A, Q3 CSD17577Q3A, Q4 CSD17577Q3A, Q5 CSD17577Q3A, U1 BQ24650, U2 BQ29700, U3 TPS61022

Commit message: Update Dynakku.kicad_pcb, Dynakku.kicad_pcb, Dynakku.kicad_prl, and 2 more files
Parts:
- moved C8 83.8 mm to (109.2, 74.8), turned to 90 degrees
- moved C10 78.8 mm to (104.8, 74.8), turned to 90 degrees
- moved C9 76.1 mm to (107.0, 74.8), turned to 90 degrees
- moved L1 73.6 mm to (101.6, 81.8), turned to 0 degrees
- moved Q2 69.8 mm to (100.0, 75.4)
- moved R5 67.8 mm to (118.5, 74.4)
- moved R6 67.1 mm to (118.5, 77.7)
- moved R7 66.4 mm to (118.5, 80.9)
- moved R9 63.0 mm to (107.8, 83.1), turned to 0 degrees
- moved C5 60.1 mm to (113.1, 74.8), turned to 90 degrees
- moved C6 58.4 mm to (123.1, 88.2)
- moved C7 58.4 mm to (123.3, 91.8)
- moved C11 57.6 mm to (107.8, 84.8), turned to 0 degrees
- moved U1 57.1 mm to (108.5, 79.6)
- moved Q3 56.0 mm to (93.5, 81.2)
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Routing:
- net /MPPT Charger/BQ24650_PH: track 0.00 -> 15.7 mm
- net +BATT: track 0.00 -> 7.85 mm
- net GND: track 0.80 -> 6.52 mm, vias 39 -> 23
- net /MPPT Charger/BQ24650_SRP: track 0.00 -> 4.71 mm
- net VDC: track 8.90 -> 13.0 mm
- net Net-(D1-K): track 27.7 -> 31.1 mm
- net /MPPT Charger/BQ24650_VFB: track 0.00 -> 1.88 mm
- net Net-(Q1-G): track 5.44 -> 7.24 mm
- net Net-(D3-K): vias 7 -> 5
- removed copper zone on B.Cu, net GND

Commit message: Update Dynakku.kicad_pcb, usb_boost.kicad_sch, Dynakku.kicad_pcb, and 3 more files
Parts:
- added JP1: SolderJumper_2_Open, Jumper:SolderJumper-2_P1.3mm_Open_RoundedPad1.0x1.5mm, B.Cu at (94.2, 104.4)
- moved R4 54.2 mm to (112.2, 81.9), turned to -90 degrees
- moved R3 53.5 mm to (112.8, 79.3)
- moved C4 47.5 mm to (113.8, 81.9), turned to -90 degrees
- moved D7 37.1 mm to (107.0, 68.8), turned to 180 degrees
- moved C7 20.8 mm to (111.2, 74.8), turned to 90 degrees
- moved C6 20.6 mm to (112.9, 70.4), turned to 90 degrees
- moved R5 14.0 mm to (111.3, 86.5), turned to 90 degrees
- moved R7 12.9 mm to (109.7, 90.3)
- moved R6 11.5 mm to (112.9, 87.8), turned to -90 degrees
- moved C3 11.1 mm to (109.4, 87.5), turned to -90 degrees
- moved J4 6.60 mm to (112.7, 96.3)
- moved J5 6.60 mm to (112.7, 91.6)
- moved R11 5.14 mm to (107.1, 89.4)
- moved C12 5.13 mm to (101.1, 87.6)
- moved C13 5.13 mm to (103.4, 87.6)
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Connections:
- U3 pad 5: +BATT -> /USB Boost/TPS_EN
Routing:
- net /MPPT Charger/BQ24650_LODRV: track 0.00 -> 15.9 mm
- net /MPPT Charger/BQ24650_BTST: track 0.00 -> 13.2 mm, vias 0 -> 2
- net /MPPT Charger/BQ24650_TS: track 0.00 -> 7.85 mm
- net /MPPT Charger/BQ24650_VFB: track 1.88 -> 8.51 mm, vias 0 -> 2
- net /MPPT Charger/BQ24650_MPPSET: track 0.00 -> 5.16 mm
- net /MPPT Charger/BQ24650_VCC: track 0.00 -> 4.47 mm
- net /MPPT Charger/BQ24650_VREF: track 0.00 -> 3.95 mm
- net GND: track 6.52 -> 10.4 mm, vias 23 -> 33
- net Net-(R6-Pad2): track 0.00 -> 2.99 mm
- net VDC: track 13.0 -> 15.9 mm
- net /MPPT Charger/BQ24650_SRP: track 4.71 -> 6.62 mm
- net +BATT: track 7.85 -> 9.57 mm
- net /MPPT Charger/BQ24650_HIDRV: track 0.00 -> 1.66 mm, vias 0 -> 1
- added copper zone on B.Cu, net /MPPT Charger/BQ24650_SRP
- added copper zone on B.Cu, net GND
- added copper zone on B.Cu, net VDC
