File: .history/usb_boost.kicad_sch (KiCad schematic)
At the start: 8 parts, among them U3 TPS61022

Commit message: Update mcp_config.json, Dynakku.kicad_pcb, Dynakku.kicad_sch, and 20 more files
Parts:
- L2: footprint (none) -> Inductor_SMD:L_Vishay_IHLP-2020
Changed lines of the file:
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@@
 			)
 		)
-		(property "Footprint" ""
+		(property "Footprint" "Inductor_SMD:L_Vishay_IHLP-2020"
 			(at 118.11 80.01 0)
 			(hide yes)

Commit message: Update Dynakku.kicad_pcb, usb_boost.kicad_sch, Dynakku.kicad_pcb, and 3 more files
Parts:
- added JP1: SolderJumper_2_Open, Jumper:SolderJumper-2_P1.3mm_Open_RoundedPad1.0x1.5mm, symbol Jumper:SolderJumper_2_Open
Connections:
- net +BATT: now also JP1.2 (B); no longer U3.5 (EN)
- new net TPS_EN: JP1.1 (A), U3.5 (EN)
Changed lines of the file:
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@@
 	(wire
 		(pts
-			(xy 210.82 82.55) (xy 210.82 80.01)
+			(xy 210.82 96.52) (xy 210.82 92.71)
 		)
 		(stroke
@@
 	(wire
 		(pts
+			(xy 210.82 80.01) (xy 210.82 82.55)
+		)
+		(stroke
+			(width 0)
+			(type default)
+		)
+	)
+	(wire
+		(pts
 			(xy 43.18 50.8) (xy 53.34 50.8)
 		)
@@
 	(wire
 		(pts
-			(xy 201.93 82.55) (xy 210.82 82.55)
+			(xy 201.93 96.52) (xy 210.82 96.52)
 		)
 		(stroke
@@
 	)
 	(label "TPS_EN"
-		(at 201.93 82.55 0)
+		(at 201.93 96.52 0)
 		(effects
 			(font
@@
 					(unit 1)
 				)
+			)
+		)
+	)
+	(symbol
+		(lib_id "Jumper:SolderJumper_2_Open")
+		(at 210.82 87.63 90)
+		(unit 1)
+		(body_style 1)
+		(exclude_from_sim no)
+		(in_bom no)
+		(on_board yes)
+		(in_pos_files yes)
+		(dnp no)
+		(fields_autoplaced yes)
+		(property "Reference" "JP1"
+			(at 213.36 86.3599 90)
+			(show_name no)
+			(do_not_autoplace no)
+			(effects
+				(font
+					(size 1.27 1.27)
+				)
+				(justify right)
+			)
+		)
+		(property "Value" "SolderJumper_2_Open"
+			(at 213.36 88.8999 90)
+			(show_name no)
+			(do_not_autoplace no)
+			(effects
+				(font
+					(size 1.27 1.27)
+				)
+				(justify right)
+			)
+		)
+		(property "Footprint" "Jumper:SolderJumper-2_P1.3mm_Open_RoundedPad1.0x1.5mm"
+			(at 210.82 87.63 0)
+			(hide yes)
+			(show_name no)
+			(do_not_autoplace no)
+			(effects
+				(font
+					(size 1.27 1.27)
+				)
+			)
+		)
+		(property "Datasheet" ""
+			(at 218.44 87.63 0)
+			(hide yes)
+			(show_name no)
+			(do_not_autoplace no)
+			(effects
+				(font
+					(size 1.27 1.27)
+				)
+			)
+		)
+		(property "Description" "Solder Jumper, 2-pole, open"
+			(at 215.9 87.63 0)
+			(hide yes)
+			(show_name no)
+			(do_not_autoplace no)
+			(effects
+				(font
+					(size 1.27 1.27)
+				)
+			)
+		)
+		(pin "2"
+		)
+		(pin "1"
+		)
+		(instances
+			(project "Dynakku"
+				(path "/ae2c3cd8-d75c-4533-b378-e05723f24e06"
+					(reference "JP1")
+					(unit 1)
+				)
